File: EurorackUtility.sch (KiCad schematic (older format))
At the start: 69 parts

Commit message: Annotated and plotted
Parts:
- gave numbers to parts that had none: 61
Connections:
- net +3V3: now also U4.1 (REF), U4.13 (VDDIO), U4.7 (VDD)
